File: left_hand/diff_i2c.kicad_sch (KiCad schematic)
At the start: 12 parts, among them J2 Conn_01x08, J3 Conn_01x03, U2 PCA9615DP

Commit message: Added current and voltage sensing on control board
Parts:
- renumbered J2 to J5, J3 to J6, R1 to R12, R2 to R13, R3 to R14, R4 to R15, R5 to R16, R6 to R17, R7 to R18, R8 to R19, U2 to U4
Changed lines of the file:
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@@
 		(dnp no)
 		(fields_autoplaced yes)
-		(property "Reference" "R4"
+		(property "Reference" "R15"
 			(at 120.65 88.8999 0)
 			(effects
@@
 			(project "left_hand"
 				(path "/22d0e2d6-ca63-4bde-b22b-39e933f56b8a/d233f6b1-7cc7-45e2-8eec-001e6bf4b7cc"
-					(reference "R4")
+					(reference "R15")
 					(unit 1)
 				)
@@
 		(dnp no)
 		(fields_autoplaced yes)
-		(property "Reference" "#PWR043"
+		(property "Reference" "#PWR048"
 			(at 182.88 95.25 0)
 			(effects
@@
 			(project "left_hand"
 				(path "/22d0e2d6-ca63-4bde-b22b-39e933f56b8a/d233f6b1-7cc7-45e2-8eec-001e6bf4b7cc"
-					(reference "#PWR043")
+					(reference "#PWR048")
 					(unit 1)
 				)
@@
 		(dnp no)
 		(fields_autoplaced yes)
-		(property "Reference" "#PWR047"
+		(property "Reference" "#PWR052"
 			(at 140.97 111.76 0)
 			(effects
@@
 			(project "left_hand"
 				(path "/22d0e2d6-ca63-4bde-b22b-39e933f56b8a/d233f6b1-7cc7-45e2-8eec-001e6bf4b7cc"
-					(reference "#PWR047")
+					(reference "#PWR052")
 					(unit 1)
 				)
@@
 		(dnp no)
 		(fields_autoplaced yes)
-		(property "Reference" "R7"
+		(property "Reference" "R18"
 			(at 185.42 114.2999 0)
 			(effects
@@
 			(project "left_hand"
 				(path "/22d0e2d6-ca63-4bde-b22b-39e933f56b8a/d233f6b1-7cc7-45e2-8eec-001e6bf4b7cc"
-					(reference "R7")
+					(reference "R18")
 					(unit 1)
 				)
@@
 		(dnp no)
 		(fields_autoplaced yes)
-		(property "Reference" "#PWR046"
+		(property "Reference" "#PWR051"
 			(at 182.88 105.41 0)
 			(effects
@@
 			(project "left_hand"
 				(path "/22d0e2d6-ca63-4bde-b22b-39e933f56b8a/d233f6b1-7cc7-45e2-8eec-001e6bf4b7cc"
-					(reference "#PWR046")
+					(reference "#PWR051")
 					(unit 1)
 				)
@@
 		(dnp no)
 		(fields_autoplaced yes)
-		(property "Reference" "R3"
+		(property "Reference" "R14"
 			(at 185.42 83.8199 0)
 			(effects
@@
 			(project "left_hand"
 				(path "/22d0e2d6-ca63-4bde-b22b-39e933f56b8a/d233f6b1-7cc7-45e2-8eec-001e6bf4b7cc"
-					(reference "R3")
+					(reference "R14")
 					(unit 1)
 				)
@@
 		(dnp no)
 		(fields_autoplaced yes)
-		(property "Reference" "#PWR042"
+		(property "Reference" "#PWR047"
 			(at 109.22 93.98 0)
 			(effects
@@
 			(project "left_hand"
 				(path "/22d0e2d6-ca63-4bde-b22b-39e933f56b8a/d233f6b1-7cc7-45e2-8eec-001e6bf4b7cc"
-					(reference "#PWR042")
+					(reference "#PWR047")
 					(unit 1)
 				)
@@
 		(dnp no)
 		(fields_autoplaced yes)
-		(property "Reference" "R1"
+		(property "Reference" "R12"
 			(at 185.42 63.4999 0)
 			(effects
@@
 			(project "left_hand"
 				(path "/22d0e2d6-ca63-4bde-b22b-39e933f56b8a/d233f6b1-7cc7-45e2-8eec-001e6bf4b7cc"
-					(reference "R1")
+					(reference "R12")
 					(unit 1)
 				)
@@
 		(dnp no)
 		(fields_autoplaced yes)
-		(property "Reference" "#PWR049"
+		(property "Reference" "#PWR054"
 			(at 182.88 135.89 0)
 			(effects
@@
 			(project "left_hand"
 				(path "/22d0e2d6-ca63-4bde-b22b-39e933f56b8a/d233f6b1-7cc7-45e2-8eec-001e6bf4b7cc"
-					(reference "#PWR049")
+					(reference "#PWR054")
 					(unit 1)
 				)
@@
 		(dnp no)
 		(fields_autoplaced yes)
-		(property "Reference" "#PWR044"
+		(property "Reference" "#PWR049"
 			(at 196.85 95.25 0)
 			(effects
@@
 			(project "left_hand"
 				(path "/22d0e2d6-ca63-4bde-b22b-39e933f56b8a/d233f6b1-7cc7-45e2-8eec-001e6bf4b7cc"
-					(reference "#PWR044")
+					(reference "#PWR049")
 					(unit 1)
 				)
@@
 		(dnp no)
 		(fields_autoplaced yes)
-		(property "Reference" "R2"
+		(property "Reference" "R13"
 			(at 185.42 73.6599 0)
 			(effects
@@
 			(project "left_hand"
 				(path "/22d0e2d6-ca63-4bde-b22b-39e933f56b8a/d233f6b1-7cc7-45e2-8eec-001e6bf4b7cc"
-					(reference "R2")
+					(reference "R13")
 					(unit 1)
 				)
@@
 		(dnp no)
 		(fields_autoplaced yes)
-		(property "Reference" "#PWR023"
+		(property "Reference" "#PWR043"
 			(at 182.88 64.77 0)
 			(effects
@@
 			(project "left_hand"
 				(path "/22d0e2d6-ca63-4bde-b22b-39e933f56b8a/d233f6b1-7cc7-45e2-8eec-001e6bf4b7cc"
-					(reference "#PWR023")
+					(reference "#PWR043")
 					(unit 1)
 				)
@@
 		(dnp no)
 		(fields_autoplaced yes)
-		(property "Reference" "#PWR037"
+		(property "Reference" "#PWR045"
 			(at 170.18 88.9 0)
 			(effects
@@
 			(project "left_hand"
 				(path "/22d0e2d6-ca63-4bde-b22b-39e933f56b8a/d233f6b1-7cc7-45e2-8eec-001e6bf4b7cc"
-					(reference "#PWR037")
+					(reference "#PWR045")
 					(unit 1)
 				)
@@
 		(dnp no)
 		(fields_autoplaced yes)
-		(property "Reference" "U2"
+		(property "Reference" "U4"
 			(at 143.1641 105.41 0)
 			(effects
@@
 			(project "left_hand"
 				(path "/22d0e2d6-ca63-4bde-b22b-39e933f56b8a/d233f6b1-7cc7-45e2-8eec-001e6bf4b7cc"
-					(reference "U2")
+					(reference "U4")
 					(unit 1)
 				)
@@
 		(dnp no)
 		(fields_autoplaced yes)
-		(property "Reference" "R5"
+		(property "Reference" "R16"
 			(at 120.65 104.1399 0)
 			(effects
@@
 			(project "left_hand"
 				(path "/22d0e2d6-ca63-4bde-b22b-39e933f56b8a/d233f6b1-7cc7-45e2-8eec-001e6bf4b7cc"
-					(reference "R5")
+					(reference "R16")
 					(unit 1)
 				)
@@
 		(dnp no)
 		(fields_autoplaced yes)
-		(property "Reference" "#PWR024"
+		(property "Reference" "#PWR044"
 			(at 139.7 85.09 0)
 			(effects
@@
 			(project "left_hand"
 				(path "/22d0e2d6-ca63-4bde-b22b-39e933f56b8a/d233f6b1-7cc7-45e2-8eec-001e6bf4b7cc"
-					(reference "#PWR024")
+					(reference "#PWR044")
 					(unit 1)
 				)
@@
 		(dnp no)
 		(fields_autoplaced yes)
-		(property "Reference" "R6"
+		(property "Reference" "R17"
 			(at 185.42 104.1399 0)
 			(effects
@@
 			(project "left_hand"
 				(path "/22d0e2d6-ca63-4bde-b22b-39e933f56b8a/d233f6b1-7cc7-45e2-8eec-001e6bf4b7cc"
-					(reference "R6")
+					(reference "R17")
 					(unit 1)
 				)
@@
 		(dnp no)
 		(fields_autoplaced yes)
-		(property "Reference" "#PWR038"
+		(property "Reference" "#PWR046"
 			(at 118.11 90.17 0)
 			(effects
@@
 			(project "left_hand"
 				(path "/22d0e2d6-ca63-4bde-b22b-39e933f56b8a/d233f6b1-7cc7-45e2-8eec-001e6bf4b7cc"
-					(reference "#PWR038")
+					(reference "#PWR046")
 					(unit 1)
 				)
@@
 		(on_board yes)
 		(dnp no)
-		(property "Reference" "J3"
+		(property "Reference" "J6"
 			(at 102.616 76.962 90)
 			(effects
@@
 			(project "left_hand"
 				(path "/22d0e2d6-ca63-4bde-b22b-39e933f56b8a/d233f6b1-7cc7-45e2-8eec-001e6bf4b7cc"
-					(reference "J3")
+					(reference "J6")
 					(unit 1)
 				)
@@
 		(dnp no)
 		(fields_autoplaced yes)
-		(property "Reference" "#PWR045"
+		(property "Reference" "#PWR050"
 			(at 196.85 105.41 0)
 			(effects
@@
 			(project "left_hand"
 				(path "/22d0e2d6-ca63-4bde-b22b-39e933f56b8a/d233f6b1-7cc7-45e2-8eec-001e6bf4b7cc"
-					(reference "#PWR045")
+					(reference "#PWR050")
 					(unit 1)
 				)
@@
 		(dnp no)
 		(fields_autoplaced yes)
-		(property "Reference" "J2"
+		(property "Reference" "J5"
 			(at 165.1 69.85 90)
 			(effects
@@
 			(project "left_hand"
 				(path "/22d0e2d6-ca63-4bde-b22b-39e933f56b8a/d233f6b1-7cc7-45e2-8eec-001e6bf4b7cc"
-					(reference "J2")
+					(reference "J5")
 					(unit 1)
 				)
@@
 		(dnp no)
 		(fields_autoplaced yes)
-		(property "Reference" "R8"
+		(property "Reference" "R19"
 			(at 185.42 124.4599 0)
 			(effects
@@
 			(project "left_hand"
 				(path "/22d0e2d6-ca63-4bde-b22b-39e933f56b8a/d233f6b1-7cc7-45e2-8eec-001e6bf4b7cc"
-					(reference "R8")
+					(reference "R19")
 					(unit 1)
 				)
@@
 		(dnp no)
 		(fields_autoplaced yes)
-		(property "Reference" "#PWR048"
+		(property "Reference" "#PWR053"
 			(at 118.11 105.41 0)
 			(effects
@@
 			(project "left_hand"
 				(path "/22d0e2d6-ca63-4bde-b22b-39e933f56b8a/d233f6b1-7cc7-45e2-8eec-001e6bf4b7cc"
-					(reference "#PWR048")
-					(unit 1)
-				)
+					(reference "#PWR053")
+					(unit 1)
+				)

Commit message: Added screw terminals etc for both stepper drivers
Parts:
- renumbered J5 to J7, J6 to J8, R12 to R13, R13 to R14, R14 to R15, R15 to R16, R16 to R17, R17 to R18, R18 to R19, R19 to R20, U4 to U3
Changed lines of the file:
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@@
 		(dnp no)
 		(fields_autoplaced yes)
-		(property "Reference" "R15"
+		(property "Reference" "R16"
 			(at 120.65 88.8999 0)
 			(effects
@@
 			(project "left_hand"
 				(path "/22d0e2d6-ca63-4bde-b22b-39e933f56b8a/d233f6b1-7cc7-45e2-8eec-001e6bf4b7cc"
-					(reference "R15")
+					(reference "R16")
 					(unit 1)
 				)
@@
 		(dnp no)
 		(fields_autoplaced yes)
-		(property "Reference" "#PWR048"
+		(property "Reference" "#PWR051"
 			(at 182.88 95.25 0)
 			(effects
@@
 			(project "left_hand"
 				(path "/22d0e2d6-ca63-4bde-b22b-39e933f56b8a/d233f6b1-7cc7-45e2-8eec-001e6bf4b7cc"
-					(reference "#PWR048")
+					(reference "#PWR051")
 					(unit 1)
 				)
@@
 		(dnp no)
 		(fields_autoplaced yes)
-		(property "Reference" "#PWR052"
+		(property "Reference" "#PWR055"
 			(at 140.97 111.76 0)
 			(effects
@@
 			(project "left_hand"
 				(path "/22d0e2d6-ca63-4bde-b22b-39e933f56b8a/d233f6b1-7cc7-45e2-8eec-001e6bf4b7cc"
-					(reference "#PWR052")
+					(reference "#PWR055")
 					(unit 1)
 				)
@@
 		(dnp no)
 		(fields_autoplaced yes)
-		(property "Reference" "R18"
+		(property "Reference" "R19"
 			(at 185.42 114.2999 0)
 			(effects
@@
 			(project "left_hand"
 				(path "/22d0e2d6-ca63-4bde-b22b-39e933f56b8a/d233f6b1-7cc7-45e2-8eec-001e6bf4b7cc"
-					(reference "R18")
+					(reference "R19")
 					(unit 1)
 				)
@@
 		(dnp no)
 		(fields_autoplaced yes)
-		(property "Reference" "#PWR051"
+		(property "Reference" "#PWR054"
 			(at 182.88 105.41 0)
 			(effects
@@
 			(project "left_hand"
 				(path "/22d0e2d6-ca63-4bde-b22b-39e933f56b8a/d233f6b1-7cc7-45e2-8eec-001e6bf4b7cc"
-					(reference "#PWR051")
+					(reference "#PWR054")
 					(unit 1)
 				)
@@
 		(dnp no)
 		(fields_autoplaced yes)
-		(property "Reference" "R14"
+		(property "Reference" "R15"
 			(at 185.42 83.8199 0)
 			(effects
@@
 			(project "left_hand"
 				(path "/22d0e2d6-ca63-4bde-b22b-39e933f56b8a/d233f6b1-7cc7-45e2-8eec-001e6bf4b7cc"
-					(reference "R14")
+					(reference "R15")
 					(unit 1)
 				)
@@
 		(dnp no)
 		(fields_autoplaced yes)
-		(property "Reference" "#PWR047"
+		(property "Reference" "#PWR050"
 			(at 109.22 93.98 0)
 			(effects
@@
 			(project "left_hand"
 				(path "/22d0e2d6-ca63-4bde-b22b-39e933f56b8a/d233f6b1-7cc7-45e2-8eec-001e6bf4b7cc"
-					(reference "#PWR047")
+					(reference "#PWR050")
 					(unit 1)
 				)
@@
 		(dnp no)
 		(fields_autoplaced yes)
-		(property "Reference" "R12"
+		(property "Reference" "R13"
 			(at 185.42 63.4999 0)
 			(effects
@@
 			(project "left_hand"
 				(path "/22d0e2d6-ca63-4bde-b22b-39e933f56b8a/d233f6b1-7cc7-45e2-8eec-001e6bf4b7cc"
-					(reference "R12")
+					(reference "R13")
 					(unit 1)
 				)
@@
 		(dnp no)
 		(fields_autoplaced yes)
-		(property "Reference" "#PWR054"
+		(property "Reference" "#PWR057"
 			(at 182.88 135.89 0)
 			(effects
@@
 			(project "left_hand"
 				(path "/22d0e2d6-ca63-4bde-b22b-39e933f56b8a/d233f6b1-7cc7-45e2-8eec-001e6bf4b7cc"
-					(reference "#PWR054")
+					(reference "#PWR057")
 					(unit 1)
 				)
@@
 		(dnp no)
 		(fields_autoplaced yes)
-		(property "Reference" "#PWR049"
+		(property "Reference" "#PWR052"
 			(at 196.85 95.25 0)
 			(effects
@@
 			(project "left_hand"
 				(path "/22d0e2d6-ca63-4bde-b22b-39e933f56b8a/d233f6b1-7cc7-45e2-8eec-001e6bf4b7cc"
-					(reference "#PWR049")
+					(reference "#PWR052")
 					(unit 1)
 				)
@@
 		(dnp no)
 		(fields_autoplaced yes)
-		(property "Reference" "R13"
+		(property "Reference" "R14"
 			(at 185.42 73.6599 0)
 			(effects
@@
 			(project "left_hand"
 				(path "/22d0e2d6-ca63-4bde-b22b-39e933f56b8a/d233f6b1-7cc7-45e2-8eec-001e6bf4b7cc"
-					(reference "R13")
+					(reference "R14")
 					(unit 1)
 				)
@@
 		(dnp no)
 		(fields_autoplaced yes)
-		(property "Reference" "#PWR043"
+		(property "Reference" "#PWR046"
 			(at 182.88 64.77 0)
 			(effects
@@
 			(project "left_hand"
 				(path "/22d0e2d6-ca63-4bde-b22b-39e933f56b8a/d233f6b1-7cc7-45e2-8eec-001e6bf4b7cc"
-					(reference "#PWR043")
+					(reference "#PWR046")
 					(unit 1)
 				)
@@
 		(dnp no)
 		(fields_autoplaced yes)
-		(property "Reference" "#PWR045"
+		(property "Reference" "#PWR048"
 			(at 170.18 88.9 0)
 			(effects
@@
 			(project "left_hand"
 				(path "/22d0e2d6-ca63-4bde-b22b-39e933f56b8a/d233f6b1-7cc7-45e2-8eec-001e6bf4b7cc"
-					(reference "#PWR045")
+					(reference "#PWR048")
 					(unit 1)
 				)
@@
 		(dnp no)
 		(fields_autoplaced yes)
-		(property "Reference" "U4"
+		(property "Reference" "U3"
 			(at 143.1641 105.41 0)
 			(effects
@@
 			(project "left_hand"
 				(path "/22d0e2d6-ca63-4bde-b22b-39e933f56b8a/d233f6b1-7cc7-45e2-8eec-001e6bf4b7cc"
-					(reference "U4")
+					(reference "U3")
 					(unit 1)
 				)
@@
 		(dnp no)
 		(fields_autoplaced yes)
-		(property "Reference" "R16"
+		(property "Reference" "R17"
 			(at 120.65 104.1399 0)
 			(effects
@@
 			(project "left_hand"
 				(path "/22d0e2d6-ca63-4bde-b22b-39e933f56b8a/d233f6b1-7cc7-45e2-8eec-001e6bf4b7cc"
-					(reference "R16")
+					(reference "R17")
 					(unit 1)
 				)
@@
 		(dnp no)
 		(fields_autoplaced yes)
-		(property "Reference" "#PWR044"
+		(property "Reference" "#PWR047"
 			(at 139.7 85.09 0)
 			(effects
@@
 			(project "left_hand"
 				(path "/22d0e2d6-ca63-4bde-b22b-39e933f56b8a/d233f6b1-7cc7-45e2-8eec-001e6bf4b7cc"
-					(reference "#PWR044")
+					(reference "#PWR047")
 					(unit 1)
 				)
@@
 		(dnp no)
 		(fields_autoplaced yes)
-		(property "Reference" "R17"
+		(property "Reference" "R18"
 			(at 185.42 104.1399 0)
 			(effects
@@
 			(project "left_hand"
 				(path "/22d0e2d6-ca63-4bde-b22b-39e933f56b8a/d233f6b1-7cc7-45e2-8eec-001e6bf4b7cc"
-					(reference "R17")
+					(reference "R18")
 					(unit 1)
 				)
@@
 		(dnp no)
 		(fields_autoplaced yes)
-		(property "Reference" "#PWR046"
+		(property "Reference" "#PWR049"
 			(at 118.11 90.17 0)
 			(effects
@@
 			(project "left_hand"
 				(path "/22d0e2d6-ca63-4bde-b22b-39e933f56b8a/d233f6b1-7cc7-45e2-8eec-001e6bf4b7cc"
-					(reference "#PWR046")
+					(reference "#PWR049")
 					(unit 1)
 				)
@@
 		(on_board yes)
 		(dnp no)
-		(property "Reference" "J6"
+		(property "Reference" "J8"
 			(at 102.616 76.962 90)
 			(effects
@@
 			(project "left_hand"
 				(path "/22d0e2d6-ca63-4bde-b22b-39e933f56b8a/d233f6b1-7cc7-45e2-8eec-001e6bf4b7cc"
-					(reference "J6")
+					(reference "J8")
 					(unit 1)
 				)
@@
 		(dnp no)
 		(fields_autoplaced yes)
-		(property "Reference" "#PWR050"
+		(property "Reference" "#PWR053"
 			(at 196.85 105.41 0)
 			(effects
@@
 			(project "left_hand"
 				(path "/22d0e2d6-ca63-4bde-b22b-39e933f56b8a/d233f6b1-7cc7-45e2-8eec-001e6bf4b7cc"
-					(reference "#PWR050")
+					(reference "#PWR053")
 					(unit 1)
 				)
@@
 		(dnp no)
 		(fields_autoplaced yes)
-		(property "Reference" "J5"
+		(property "Reference" "J7"
 			(at 165.1 69.85 90)
 			(effects
@@
 			(project "left_hand"
 				(path "/22d0e2d6-ca63-4bde-b22b-39e933f56b8a/d233f6b1-7cc7-45e2-8eec-001e6bf4b7cc"
-					(reference "J5")
+					(reference "J7")
 					(unit 1)
 				)
@@
 		(dnp no)
 		(fields_autoplaced yes)
-		(property "Reference" "R19"
+		(property "Reference" "R20"
 			(at 185.42 124.4599 0)
 			(effects
@@
 			(project "left_hand"
 				(path "/22d0e2d6-ca63-4bde-b22b-39e933f56b8a/d233f6b1-7cc7-45e2-8eec-001e6bf4b7cc"
-					(reference "R19")
+					(reference "R20")
 					(unit 1)
 				)
@@
 		(dnp no)
 		(fields_autoplaced yes)
-		(property "Reference" "#PWR053"
+		(property "Reference" "#PWR056"
 			(at 118.11 105.41 0)
 			(effects
@@
 			(project "left_hand"
 				(path "/22d0e2d6-ca63-4bde-b22b-39e933f56b8a/d233f6b1-7cc7-45e2-8eec-001e6bf4b7cc"
-					(reference "#PWR053")
-					(unit 1)
-				)
+					(reference "#PWR056")
+					(unit 1)
+				)

Commit message: Started layout of control board
Parts:
- renumbered R13 to R14, R14 to R15, R15 to R16, R16 to R17, R17 to R18, R18 to R19, R19 to R20, R20 to R21
Changed lines of the file:
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@@
 		(dnp no)
 		(fields_autoplaced yes)
-		(property "Reference" "R16"
+		(property "Reference" "R17"
 			(at 120.65 88.8999 0)
 			(effects
@@
 			(project "left_hand"
 				(path "/22d0e2d6-ca63-4bde-b22b-39e933f56b8a/d233f6b1-7cc7-45e2-8eec-001e6bf4b7cc"
-					(reference "R16")
+					(reference "R17")
 					(unit 1)
 				)
@@
 		(dnp no)
 		(fields_autoplaced yes)
-		(property "Reference" "#PWR051"
+		(property "Reference" "#PWR052"
 			(at 182.88 95.25 0)
 			(effects
@@
 			(project "left_hand"
 				(path "/22d0e2d6-ca63-4bde-b22b-39e933f56b8a/d233f6b1-7cc7-45e2-8eec-001e6bf4b7cc"
-					(reference "#PWR051")
+					(reference "#PWR052")
 					(unit 1)
 				)
@@
 		(dnp no)
 		(fields_autoplaced yes)
-		(property "Reference" "#PWR055"
+		(property "Reference" "#PWR056"
 			(at 140.97 111.76 0)
 			(effects
@@
 			(project "left_hand"
 				(path "/22d0e2d6-ca63-4bde-b22b-39e933f56b8a/d233f6b1-7cc7-45e2-8eec-001e6bf4b7cc"
-					(reference "#PWR055")
+					(reference "#PWR056")
 					(unit 1)
 				)
@@
 		(dnp no)
 		(fields_autoplaced yes)
-		(property "Reference" "R19"
+		(property "Reference" "R20"
 			(at 185.42 114.2999 0)
 			(effects
@@
 			(project "left_hand"
 				(path "/22d0e2d6-ca63-4bde-b22b-39e933f56b8a/d233f6b1-7cc7-45e2-8eec-001e6bf4b7cc"
-					(reference "R19")
+					(reference "R20")
 					(unit 1)
 				)
@@
 		(dnp no)
 		(fields_autoplaced yes)
-		(property "Reference" "#PWR054"
+		(property "Reference" "#PWR055"
 			(at 182.88 105.41 0)
 			(effects
@@
 			(project "left_hand"
 				(path "/22d0e2d6-ca63-4bde-b22b-39e933f56b8a/d233f6b1-7cc7-45e2-8eec-001e6bf4b7cc"
-					(reference "#PWR054")
+					(reference "#PWR055")
 					(unit 1)
 				)
@@
 		(dnp no)
 		(fields_autoplaced yes)
-		(property "Reference" "R15"
+		(property "Reference" "R16"
 			(at 185.42 83.8199 0)
 			(effects
@@
 			(project "left_hand"
 				(path "/22d0e2d6-ca63-4bde-b22b-39e933f56b8a/d233f6b1-7cc7-45e2-8eec-001e6bf4b7cc"
-					(reference "R15")
+					(reference "R16")
 					(unit 1)
 				)
@@
 		(dnp no)
 		(fields_autoplaced yes)
-		(property "Reference" "#PWR050"
+		(property "Reference" "#PWR051"
 			(at 109.22 93.98 0)
 			(effects
@@
 			(project "left_hand"
 				(path "/22d0e2d6-ca63-4bde-b22b-39e933f56b8a/d233f6b1-7cc7-45e2-8eec-001e6bf4b7cc"
-					(reference "#PWR050")
+					(reference "#PWR051")
 					(unit 1)
 				)
@@
 		(dnp no)
 		(fields_autoplaced yes)
-		(property "Reference" "R13"
+		(property "Reference" "R14"
 			(at 185.42 63.4999 0)
 			(effects
@@
 			(project "left_hand"
 				(path "/22d0e2d6-ca63-4bde-b22b-39e933f56b8a/d233f6b1-7cc7-45e2-8eec-001e6bf4b7cc"
-					(reference "R13")
+					(reference "R14")
 					(unit 1)
 				)
@@
 		(dnp no)
 		(fields_autoplaced yes)
-		(property "Reference" "#PWR057"
+		(property "Reference" "#PWR058"
 			(at 182.88 135.89 0)
 			(effects
@@
 			(project "left_hand"
 				(path "/22d0e2d6-ca63-4bde-b22b-39e933f56b8a/d233f6b1-7cc7-45e2-8eec-001e6bf4b7cc"
-					(reference "#PWR057")
+					(reference "#PWR058")
 					(unit 1)
 				)
@@
 		(dnp no)
 		(fields_autoplaced yes)
-		(property "Reference" "#PWR052"
+		(property "Reference" "#PWR053"
 			(at 196.85 95.25 0)
 			(effects
@@
 			(project "left_hand"
 				(path "/22d0e2d6-ca63-4bde-b22b-39e933f56b8a/d233f6b1-7cc7-45e2-8eec-001e6bf4b7cc"
-					(reference "#PWR052")
+					(reference "#PWR053")
 					(unit 1)
 				)
@@
 		(dnp no)
 		(fields_autoplaced yes)
-		(property "Reference" "R14"
+		(property "Reference" "R15"
 			(at 185.42 73.6599 0)
 			(effects
@@
 			(project "left_hand"
 				(path "/22d0e2d6-ca63-4bde-b22b-39e933f56b8a/d233f6b1-7cc7-45e2-8eec-001e6bf4b7cc"
-					(reference "R14")
+					(reference "R15")
 					(unit 1)
 				)
@@
 		(dnp no)
 		(fields_autoplaced yes)
-		(property "Reference" "#PWR046"
+		(property "Reference" "#PWR047"
 			(at 182.88 64.77 0)
 			(effects
@@
 			(project "left_hand"
 				(path "/22d0e2d6-ca63-4bde-b22b-39e933f56b8a/d233f6b1-7cc7-45e2-8eec-001e6bf4b7cc"
-					(reference "#PWR046")
+					(reference "#PWR047")
 					(unit 1)
 				)
@@
 		(dnp no)
 		(fields_autoplaced yes)
-		(property "Reference" "#PWR048"
+		(property "Reference" "#PWR049"
 			(at 170.18 88.9 0)
 			(effects
@@
 			(project "left_hand"
 				(path "/22d0e2d6-ca63-4bde-b22b-39e933f56b8a/d233f6b1-7cc7-45e2-8eec-001e6bf4b7cc"
-					(reference "#PWR048")
+					(reference "#PWR049")
 					(unit 1)
 				)
@@
 		(dnp no)
 		(fields_autoplaced yes)
-		(property "Reference" "R17"
+		(property "Reference" "R18"
 			(at 120.65 104.1399 0)
 			(effects
@@
 			(project "left_hand"
 				(path "/22d0e2d6-ca63-4bde-b22b-39e933f56b8a/d233f6b1-7cc7-45e2-8eec-001e6bf4b7cc"
-					(reference "R17")
+					(reference "R18")
 					(unit 1)
 				)
@@
 		(dnp no)
 		(fields_autoplaced yes)
-		(property "Reference" "#PWR047"
+		(property "Reference" "#PWR048"
 			(at 139.7 85.09 0)
 			(effects
@@
 			(project "left_hand"
 				(path "/22d0e2d6-ca63-4bde-b22b-39e933f56b8a/d233f6b1-7cc7-45e2-8eec-001e6bf4b7cc"
-					(reference "#PWR047")
+					(reference "#PWR048")
 					(unit 1)
 				)
@@
 		(dnp no)
 		(fields_autoplaced yes)
-		(property "Reference" "R18"
+		(property "Reference" "R19"
 			(at 185.42 104.1399 0)
 			(effects
@@
 			(project "left_hand"
 				(path "/22d0e2d6-ca63-4bde-b22b-39e933f56b8a/d233f6b1-7cc7-45e2-8eec-001e6bf4b7cc"
-					(reference "R18")
+					(reference "R19")
 					(unit 1)
 				)
@@
 		(dnp no)
 		(fields_autoplaced yes)
-		(property "Reference" "#PWR049"
+		(property "Reference" "#PWR050"
 			(at 118.11 90.17 0)
 			(effects
@@
 			(project "left_hand"
 				(path "/22d0e2d6-ca63-4bde-b22b-39e933f56b8a/d233f6b1-7cc7-45e2-8eec-001e6bf4b7cc"
-					(reference "#PWR049")
+					(reference "#PWR050")
 					(unit 1)
 				)
@@
 		(dnp no)
 		(fields_autoplaced yes)
-		(property "Reference" "#PWR053"
+		(property "Reference" "#PWR054"
 			(at 196.85 105.41 0)
 			(effects
@@
 			(project "left_hand"
 				(path "/22d0e2d6-ca63-4bde-b22b-39e933f56b8a/d233f6b1-7cc7-45e2-8eec-001e6bf4b7cc"
-					(reference "#PWR053")
+					(reference "#PWR054")
 					(unit 1)
 				)
@@
 		(dnp no)
 		(fields_autoplaced yes)
-		(property "Reference" "R20"
+		(property "Reference" "R21"
 			(at 185.42 124.4599 0)
 			(effects
@@
 			(project "left_hand"
 				(path "/22d0e2d6-ca63-4bde-b22b-39e933f56b8a/d233f6b1-7cc7-45e2-8eec-001e6bf4b7cc"
-					(reference "R20")
+					(reference "R21")
 					(unit 1)
 				)
@@
 		(dnp no)
 		(fields_autoplaced yes)
-		(property "Reference" "#PWR056"
+		(property "Reference" "#PWR057"
 			(at 118.11 105.41 0)
 			(effects
@@
 			(project "left_hand"
 				(path "/22d0e2d6-ca63-4bde-b22b-39e933f56b8a/d233f6b1-7cc7-45e2-8eec-001e6bf4b7cc"
-					(reference "#PWR056")
-					(unit 1)
-				)
+					(reference "#PWR057")
+					(unit 1)
+				)
