File: v2/control_pcb/current_sensing.kicad_sch (KiCad schematic)
At the start: 20 parts, among them J14 Conn_02x02_Top_Bottom, J15 Conn_02x02_Top_Bottom, U10 TMCS1108A3UQDR, U11 TMCS1108A3UQDR, U6 TMCS1108A3UQDR, U7 TMCS1108A3UQDR, U8 ADS7828, U9 LM4040LP-4.1

Commit message: Doing stuff
Parts:
- removed C6, C7: 0.1uF, Capacitor_THT:C_Rect_L4.6mm_W2.0mm_P2.50mm_MKS02_FKP02, symbol Device:C
- removed C8: 1uF, Capacitor_THT:C_Rect_L4.6mm_W2.0mm_P2.50mm_MKS02_FKP02, symbol Device:C
- removed R17: 904R, Resistor_THT:R_Axial_DIN0207_L6.3mm_D2.5mm_P10.16mm_Horizontal, symbol Device:R_US
- removed U8: ADS7828, Package_SO:TSSOP-16_4.4x5mm_P0.65mm, symbol Analog_ADC:ADS7828
- removed U9: LM4040LP-4.1, Package_TO_SOT_THT:TO-92_Inline, symbol Reference_Voltage:LM4040LP-4.1
Connections:
- no-connect marks 6 -> 4

Commit message: Doing some things
Crossing some ts and dotting some is. Making v3 of the BOM.
Parts:
- added C6: 0.1uF, Capacitor_THT:C_Rect_L4.6mm_W2.0mm_P2.50mm_MKS02_FKP02, symbol Device:C
- added R22, R23: 0R, Resistor_THT:R_Axial_DIN0207_L6.3mm_D2.5mm_P10.16mm_Horizontal, symbol Device:R_US
- added U9: ~, Package_DFN_QFN:WQFN-16-1EP_3x3mm_P0.5mm_EP1.68x1.68mm, symbol bh_symbol_library:ADS7138IRTER
Connections:
- net +5V: now also C6.1, U9.10 (DVDD), U9.7 (AVDD)
- net GND: now also C6.2, R23.2, U9.9 (GND)
- net at R19.2, R21.1: now also U9.4 (AIN5)
- net at U11.3 (IN-), U11.4 (IN-): now also J15.4 (Pin_4); no longer J15.3 (Pin_3)
- net at U11.7 (VOUT): now also U9.2 (AIN3)
- net at U7.3 (IN-), U7.4 (IN-): now also J14.4 (Pin_4); no longer J14.3 (Pin_3)
- net at U7.7 (VOUT): now also U9.16 (AIN1)
- net at U10.3 (IN-), U10.4 (IN-): now also J15.3 (Pin_3); no longer J15.4 (Pin_4)
- net at U6.3 (IN-), U6.4 (IN-): now also J14.3 (Pin_3); no longer J14.4 (Pin_4)
- net at U6.7 (VOUT): now also U9.15 (AIN0)
- net at U10.7 (VOUT): now also U9.1 (AIN2)
- net at R18.2, R20.1: now also U9.3 (AIN4)
- new net: R22.1, U9.8 (DECAP)
- new net: R22.2, R23.1, U9.11 (ADDR)
- new net SCL: U9.13 (SCL)
- new net SDA: U9.14 (SDA)
- no-connect marks 4 -> 7

Commit message: Doing more things
Parts:
- removed R20: 4k, Resistor_THT:R_Axial_DIN0207_L6.3mm_D2.5mm_P10.16mm_Horizontal, symbol Device:R_US
- added R17: 4k, Resistor_THT:R_Axial_DIN0207_L6.3mm_D2.5mm_P10.16mm_Horizontal, symbol Device:R_US
- U9: value ~ -> ADS7138IRTER
Connections:
- net +12V: now also U10.1 (IN+), U10.2 (IN+), U6.1 (IN+), U6.2 (IN+); no longer U11.1 (IN+), U11.2 (IN+), U7.1 (IN+), U7.2 (IN+)
- net +5V: now also U11.1 (IN+), U11.2 (IN+), U7.1 (IN+), U7.2 (IN+), U9.3 (AIN4); no longer R18.1, U10.1 (IN+), U10.2 (IN+), U6.1 (IN+), U6.2 (IN+)
- net GND: now also R18.2
- net at U9.5 (AIN6): now also R18.1, R17.2
- new net +24V: R17.1
- no-connect marks 7 -> 6
Other:
- note added: "ADC"
- note removed: "ADC AND VOLTAGE SENSING"
