File: v2/control_pcb/control_pcb.kicad_sch (KiCad schematic)
At the start: 27 parts, among them J1 Raspberry_Pi_2_3, J10 8P8C_Shielded, J11 Screw_Terminal_01x02, J12 Screw_Terminal_01x02, J13 Screw_Terminal_01x02, J2 8P8C_Shielded, J6 Screw_Terminal_01x02, J7 Screw_Terminal_01x02, J8 Screw_Terminal_01x08, J9 Screw_Terminal_01x08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

Commit message: Doing more things 2
Other:
- note added: "BOT-HOVEN Control PCB Version 2"
- note added: "Drawn: Jascha Petersen"
- note added: "I2C LEVEL SHIFTER"
- note added: "RASPBERRY PI"
- note added: "RASPBERRY PI PICO"
Changed lines of the file:
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@@
+		)
+	)
+	(text "BOT-HOVEN Control PCB Version 2\n"
+		(exclude_from_sim no)
+		(at 217.678 168.91 0)
+		(effects
+			(font
+				(size 3 3)
+				(thickness 0.6)
+				(bold yes)
+			)
 		)
 	)
@@
 		(effects
 			(font
+				(size 2 2)
+			)
+		)
+	)
+	(text "I2C LEVEL SHIFTER"
+		(exclude_from_sim no)
+		(at 92.964 24.892 0)
+		(effects
+			(font
+				(size 2 2)
+			)
+		)
+	)
+	(text "Drawn: Jascha Petersen"
+		(exclude_from_sim no)
+		(at 195.58 179.832 0)
+		(effects
+			(font
+				(size 2 2)
+			)
+		)
+	)
+	(text "RASPBERRY PI\nPICO\n"
+		(exclude_from_sim no)
+		(at 165.862 30.226 0)
+		(effects
+			(font
+				(size 2 2)
+			)
+		)
+	)
+	(text "RASPBERRY PI"
+		(exclude_from_sim no)
+		(at 26.416 15.748 0)
+		(effects
+			(font
